File: design_files/ASM2027-Rev3.brd (EAGLE design)
At the start: 30 x 30 mm, 80 parts, among them J1 47346-0001, J10 SM03B-SRSS-TB, J11 SM05B, J12 SM05B, J13 SM05B, J14 SM05B, J15 SM03B-SRSS-TB, J16 SM03B-SRSS-TB, J17 SM03B-SRSS-TB, J2 SM02B-SRSS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

Commit message: dc motor updates
Parts:
- C3: value 47uF -> 10uF
- SW3: device tinycircuits:KXT_LHS_1 -> tinycircuits:KXT_LHS
Connections:
- net IO31: no longer U5.12, U7.12
- net N$24: now also U5.12
- net N$41: now also U7.12
Routing:
- net IO31: track 28.2 -> 7.31 mm, vias 3 -> 0
- net N$41: track 1.83 -> 9.18 mm, vias 0 -> 2
- net N$24: track 3.38 -> 9.17 mm, vias 1 -> 2
- net IO26: track 33.7 -> 32.9 mm
- net GND: track 71.1 -> 70.4 mm
- net VBATT: track 92.4 -> 93.1 mm
- net CE: track 25.9 -> 26.5 mm
Other:
- board text added: "ASM2027 Rev3"
- board text removed: "4"
- board text removed: "ASM2027 Rev4"
