File: design_files/ASM2027-Rev3.sch (EAGLE design)
At the start: 79 parts, among them J1 47346-0001, J10 SM03B-SRSS-TB, J11 SM05B, J12 SM05B, J13 SM05B, J14 SM05B, J15 SM03B-SRSS-TB, J16 SM03B-SRSS-TB, J17 SM03B-SRSS-TB, J2 SM02B-SRSS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

Commit message: dc motor updates
Parts:
- C3: value 47uF -> 10uF; device tinycircuits:AS-ITM-00558 -> tinycircuits:AS-ITM-00002; PARTNO AS-ITM-00558 -> AS-ITM-00002; VALUE 47uF -> (none)
- SW3: device tinycircuits:AS-ITM-003721 -> tinycircuits:AS-ITM-00372
Connections:
- net IO31: no longer U5.CONFIG, U7.CONFIG
- net N$24: now also U5.CONFIG
- net N$41: now also U7.CONFIG
Other:
- note added: "3"
- note removed: "4"
